File: vl670.kicad_pcb (KiCad board)
At the start: 4 copper layers, 65 x 35 mm, 119 parts, among them J1 Conn_01x07_Male, J2 USB_C_Receptacle, J3 Conn_01x08_Male, J4 USB3_A Receptacle, J5 Conn_01x02_Male, U1 HD3SS3220, U2 VL670, U3 74LVC2G66, U4 TPS2061C-PXLI, U5 74LVC2G66, U6 GD25D05, Y1 25MHz

Commit message: usb-b edition
Parts:
- removed C12: 1uF, Capacitor_SMD:C_0603_1608Metric_Pad1.08x0.95mm_HandSolder
- removed C25: 470nF, Capacitor_SMD:C_0603_1608Metric_Pad1.08x0.95mm_HandSolder
- removed C3, C4, C5, C6: 220nF, Capacitor_SMD:C_0603_1608Metric_Pad1.08x0.95mm_HandSolder
- removed D5: ESD7104, vl670:OnSemi_UDFN-10_1.0x2.5mm_P0.5mm
- removed R12, R18: 1.8M, Resistor_SMD:R_0603_1608Metric_Pad0.98x0.95mm_HandSolder
- removed R14: 200k, Resistor_SMD:R_0603_1608Metric_Pad0.98x0.95mm_HandSolder
- removed R16, R17: 100K, Resistor_SMD:R_0402_1005Metric_Pad0.72x0.64mm_HandSolder
- removed U1: HD3SS3220, vl670:Texas_VQFN-RNH-30
- D10, D11, D12, D13, D15, D16, D17, D19, D8, D9: value ESD7951S -> ESD5B5.0ST1G-N
- FB1: value Ferrite_Bead_Small -> BLM18KG221SN1D
- J2: value USB_C_Receptacle -> USB3_B; footprint vl670:USB_C_Receptacle_XKB_U262-241N-4BV60 -> vl670:USB3_B_XKB_U235-091N-4BLRC16-4-5
- moved C79 25.0 mm to (196.2, 135.1), turned to 0 degrees
- moved C81 21.6 mm to (198.5, 131.0), turned to 180 degrees
- moved C80 21.1 mm to (196.2, 133.1), turned to 0 degrees
- moved C82 18.3 mm to (198.5, 132.4), turned to 180 degrees
- moved D1 16.9 mm to (184.0, 133.0)
- moved C1 15.3 mm to (195.6, 128.5), turned to 180 degrees
- moved C2 15.3 mm to (195.6, 130.0), turned to 180 degrees
- moved R2 15.2 mm to (195.6, 134.8)
- moved FB1 14.9 mm to (188.7, 133.4)
- moved R1 13.0 mm to (195.6, 133.3)
- moved JP2 12.9 mm to (190.1, 130.9)
- moved D4 12.3 mm to (190.2, 123.2), turned to 0 degrees
- moved J2 7.79 mm to (183.0, 122.0), turned to 0 degrees
- moved TP3 7.50 mm to (206.8, 133.0)
- moved C73 6.79 mm to (190.7, 127.0), turned to 0 degrees
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Connections:
- net /D_DEMUX+ renamed /D_DC+
- net /D_DEMUX- renamed /D_DC-
- C1 pad 1: /USB AC CAP/ESD/MUX/TX1_AC- -> /SSRX_DC-
- C1 pad 2: /USB AC CAP/ESD/MUX/TX1- -> /SSRX+
- C2 pad 1: /USB AC CAP/ESD/MUX/TX1_AC+ -> /SSRX_DC+
- C2 pad 2: /USB AC CAP/ESD/MUX/TX1+ -> /SSRX-
- D1 pad 1: /USB AC CAP/ESD/MUX/RX1+ -> /D+
- D1 pad 10: /USB AC CAP/ESD/MUX/RX1+ -> /D+
- D1 pad 2: /USB AC CAP/ESD/MUX/RX1- -> /D-
- D1 pad 4: /USB AC CAP/ESD/MUX/TX1+ -> +5VP
- D1 pad 5: /USB AC CAP/ESD/MUX/TX1- -> +5VP
- D1 pad 6: /USB AC CAP/ESD/MUX/TX1- -> +5VP
- D1 pad 7: /USB AC CAP/ESD/MUX/TX1+ -> +5VP
- D1 pad 9: /USB AC CAP/ESD/MUX/RX1- -> /D-
- D4 pad 1: /USB AC CAP/ESD/MUX/RX2- -> /SSTX+
- D4 pad 10: /USB AC CAP/ESD/MUX/RX2- -> /SSTX+
- D4 pad 2: /USB AC CAP/ESD/MUX/RX2+ -> /SSTX-
- D4 pad 4: /USB AC CAP/ESD/MUX/TX2- -> /SSRX+
- D4 pad 5: /USB AC CAP/ESD/MUX/TX2+ -> /SSRX-
- D4 pad 6: /USB AC CAP/ESD/MUX/TX2+ -> /SSRX-
- D4 pad 7: /USB AC CAP/ESD/MUX/TX2- -> /SSRX+
- D4 pad 9: /USB AC CAP/ESD/MUX/RX2+ -> /SSTX-
- FID1 pad : GND -> (no net)
- FID2 pad : GND -> (no net)
- FID3 pad : GND -> (no net)
- FID4 pad : GND -> (no net)
- FID5 pad : GND -> (no net)
- FID6 pad : GND -> (no net)
- FID7 pad : GND -> (no net)
- FID8 pad : GND -> (no net)
- R1 pad 2: /USB AC CAP/ESD/MUX/D- -> /D-
- R2 pad 2: /USB AC CAP/ESD/MUX/D+ -> /D+
- U2 pad 13: /SSTX_DEMUX+ -> /SSRX_DC-
- U2 pad 14: /SSTX_DEMUX- -> /SSRX_DC+
- U2 pad 18: /SSRX_DEMUX- -> /SSTX+
- U2 pad 19: /SSRX_DEMUX+ -> /SSTX-
Routing:
- net /USB AC CAP/ESD/MUX/CC2: track 47.0 -> 0.00 mm, vias 3 -> 0
- net /SSTX-: track 0.00 -> 32.7 mm, vias 0 -> 3
- net /SSTX+: track 0.00 -> 32.1 mm, vias 0 -> 3
- net /D+: track 0.00 -> 29.0 mm
- net /USB AC CAP/ESD/MUX/RX1-: track 28.9 -> 0.00 mm, vias 1 -> 0
- net /D-: track 0.00 -> 28.5 mm
- net /USB AC CAP/ESD/MUX/RX1+: track 28.5 -> 0.00 mm, vias 1 -> 0
- net GND: track 686.8 -> 661.8 mm, vias 172 -> 159
- net /USB AC CAP/ESD/MUX/RX2+: track 23.2 -> 0.00 mm
- net /USB AC CAP/ESD/MUX/RX2-: track 23.2 -> 0.00 mm
- net /SSRX_DEMUX+: track 22.9 -> 0.00 mm, vias 2 -> 0
- net /USB AC CAP/ESD/MUX/TX2-: track 22.8 -> 0.00 mm, vias 1 -> 0
- net /SSRX_DEMUX-: track 22.5 -> 0.00 mm, vias 2 -> 0
- net /USB AC CAP/ESD/MUX/TX2+: track 22.4 -> 0.00 mm, vias 1 -> 0
- net /D_DC+: track 38.7 -> 18.7 mm
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