File: vl670.sch (KiCad schematic (older format))
At the start: 58 parts, among them J1 Conn_01x07_Male, J2 USB_C_Receptacle, J3 Conn_01x07_Male, J4 USB3_A Receptacle, J5 Conn_01x02_Male, U2 VL670, U4 TPS2061C-PXLI, Y1 25MHz

Commit message: v0.02.
Parts:
- removed J3: Conn_01x07_Male, Connector_PinHeader_2.54mm:PinHeader_1x07_P2.54mm_Vertical, symbol Connector:Conn_01x07_Male
- added D19: ESD5B5.0ST1G-N, Diode_SMD:D_SOD-523, symbol Device:D_TVS
- added D20: LED, LED_SMD:LED_0603_1608Metric_Pad1.05x0.95mm_HandSolder, symbol Device:LED
- added FB1: BLM18KG221SN1D, Inductor_SMD:L_0603_1608Metric_Pad1.05x0.95mm_HandSolder, symbol Device:Ferrite_Bead_Small
- added J3: Conn_01x08_Male, Connector_PinHeader_2.54mm:PinHeader_1x08_P2.54mm_Vertical, symbol Connector:Conn_01x08_Male
- added R13, R24: 470R, Resistor_SMD:R_0603_1608Metric_Pad0.98x0.95mm_HandSolder, symbol Device:R_US
- added R22, R23: 0R5, Resistor_SMD:R_0603_1608Metric_Pad0.98x0.95mm_HandSolder, symbol Device:R_US
- C19, C20: value 1uF -> 10uF
- D10, D11, D12, D13, D15, D16, D17, D8, D9: value ESD7951S -> ESD5B5.0ST1G-N
Connections:
- net +5V: now also J5.1 (Pin_1); no longer J5.2 (Pin_2)
- net +5VP: now also FB1.2; no longer JP2.1 (A)
- net +5V_SW: now also D20.2 (A)
- net GND: now also J5.2 (Pin_2), D19.2 (A2), J3.8 (Pin_8), R22.2, R23.2, R24.2; no longer C19.2, C20.2, J5.1 (Pin_1)
- net at U2.36 (GPIO1_1/GPIO_TP2): now also D7.1 (A1), R9.2, J3.2 (Pin_2)
- net at D9.1 (A1), R20.1, U2.38 (GPIO1_2/GPIO_TP3): now also J3.4 (Pin_4)
- net at D8.1 (A1), R21.1, U2.39 (GPIO1_0/GPIO_TP1): now also J3.3 (Pin_3)
- net at U2.4 (GPIO3_0/STATUS): now also D19.1 (A1), J3.1 (Pin_1), R13.2; no longer R9.2
- net at D12.1 (A1), U2.45 (GPIO3_1/GPIO_TP4): now also J3.7 (Pin_7)
- net at D11.1 (A1), U2.6 (GPIO2_1/UART_TX): now also J3.6 (Pin_6)
- net at D10.1 (A1), U2.7 (GPIO2_0/UART_RX): now also J3.5 (Pin_5)
- net at D2.2 (A), R9.1: now also R13.1
- new net: C19.2, R22.1
- new net: C20.2, R23.1
- new net: FB1.1, JP2.1 (A)
- new net: D20.1 (K), R24.1
Other:
- note added: "C1+C5+C7=73 nF"
- note added: "FB1 may resonate, see\n capacitor C19, C20"
- note added: "Note:"
- note added: "On VL670, without R20,\nfirewire reads false input\nand random reset."
- note added: "R51, R52 damp FB1\ninductance resonance.\nWithout FB1, use 0R."
- note added: "VL670: R9\nVL671: R13"
- note added: "VL671: 1.2V"
- note removed: "C1//C5//C7 = 73 uF"
- note removed: "R20 is important"
- moved on the sheet: C19, C20, C7, C8, D10, D11, D12, D3, D7, D8, D9, J4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

Commit message: usb-b edition
Parts:
- removed J2: USB_C_Receptacle, vl670:USB_C_Receptacle_XKB_U262-241N-4BV60, symbol Connector:USB_C_Receptacle
- added C1, C2: 220nF, Capacitor_SMD:C_0603_1608Metric_Pad1.08x0.95mm_HandSolder, symbol Device:C_Small
- added D1, D4: ESD7104, vl670:OnSemi_UDFN-10_1.0x2.5mm_P0.5mm, symbol vl670:ESD7104
- added J2: USB3_B, vl670:USB3_B_XKB_U235-091N-4BLRC16-4-5, symbol Connector:USB3_B
Connections:
- net +5VP: now also D1.4 (TVS3), D1.5 (TVS4), D1.6 (NC4), D1.7 (NC3), J2.1 (VBUS)
- net GND: now also D1.3 (COM), D1.8 (GND), D4.3 (COM), D4.8 (GND), J2.10 (SHIELD), J2.4 (GND), J2.7 (DRAIN)
- net D_DEMUX+ renamed D_DC+
- net D_DEMUX- renamed D_DC-
- net SSRX_DEMUX+ renamed SSTX+
- net SSTX+: now also D4.1 (TVS1), D4.10 (NC1), J2.6 (SSTX+)
- net SSRX_DEMUX- renamed SSTX-
- net SSTX-: now also D4.2 (TVS2), D4.9 (NC2), J2.5 (SSTX-)
- net SSTX_DEMUX+ renamed SSRX_DC-
- net SSRX_DC-: now also C1.1
- net SSTX_DEMUX- renamed SSRX_DC+
- net SSRX_DC+: now also C2.1
- net USB AC CAP/ESD/MUX/D+ renamed D+
- net D+: now also D1.1 (TVS1), D1.10 (NC1), J2.3 (D+)
- net USB AC CAP/ESD/MUX/D- renamed D-
- net D-: now also D1.2 (TVS2), D1.9 (NC2), J2.2 (D-)
- new net SSRX+: C2.2, D4.4 (TVS3), D4.7 (NC3), J2.9 (SSRX+)
- new net SSRX-: C1.2, D4.5 (TVS4), D4.6 (NC4), J2.8 (SSRX-)
- no-connect marks 3 -> 1
Other:
- note added: "C1+C7=110nF"
- note removed: "C1+C5+C7=73 nF"
- moved on the sheet: FB1, JP2
